File: Kicad/512K ISA/512k.kicad_pcb (KiCad board)
At the start: 2 copper layers, 104 x 73.9 mm, 15 parts, among them J9 Bus_ISA_8bit, U1 62256, U2 28C256, U3 AS6C4008, U4 74LS139, U5 74LS138

Commit message: Updated Kicad files
Other:
- board text added: "EMM COMPUTERS 512K RAM, 32K ROM/RAM Copyright (C) 2022 EMM www.homebrew8088.com"
- board text removed: "EMM COMPUTERS 512K RAM, 32K ROM/RAM Copyright (C) 2021 EMM www.homebrew8088.com"
