File: Kicad/Multi ATX 4 ISA/Multi.sch (KiCad schematic (older format))
At the start: 65 parts, among them J1 Bus_ISA_8bit, J10 Conn_02x08_Counter_Clockwise, J2 Mini-DIN-6, J3 SPK, J5 IRQ6 EN, J6 PWR ON, J7 Bus_ISA_8bit, J8 Bus_ISA_8bit, J9 Bus_ISA_8bit, SW1 RESET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

Commit message: Added port 0x61 read to 4 slot main board
Parts:
- removed J5: IRQ6 EN, Connector_PinHeader_2.54mm:PinHeader_1x02_P2.54mm_Vertical, symbol Connector_Generic:Conn_01x02
- removed R10, R11, R15: 10k ohm, Resistor_THT:R_Axial_DIN0207_L6.3mm_D2.5mm_P10.16mm_Horizontal, symbol Device:R
- added C11, C13: 0.1uF, Capacitor_THT:C_Disc_D4.3mm_W1.9mm_P5.00mm, symbol pspice:CAP
- added RN3: 10k ohm, Resistor_THT:R_Array_SIP4, symbol Device:R_Network03
- added U1: 74LS139, Package_DIP:DIP-16_W7.62mm, symbol 74xx:74LS139
- added U2: 74LS245, Package_DIP:DIP-20_W7.62mm, symbol 74xx:74LS245
Connections:
- net 5+: now also C11.2, C13.2, U1.16 (VCC), U2.20 (VCC)
- net D0: now also U2.9 (A7)
- net D1: now also U2.8 (A6)
- net D2: now also U2.7 (A5)
- net D3: now also U2.6 (A4)
- net D4: now also U2.5 (A3)
- net D5: now also U2.4 (A2)
- net D6: now also U2.3 (A1)
- net D7: now also U2.2 (A0)
- net DRQ0: now also RN3.4 (R3)
- net GND: now also C11.1, C13.1, RN3.1 (common), U1.13 (A1), U1.3 (A1), U1.8 (GND), U2.1 (A->B), U2.10 (GND); no longer U117.3 (A1)
- net HOLD: now also RN3.3 (R2)
- net IN_IRQ6: no longer U16.13
- net IORD: now also U1.14 (A0)
- net IOWR: now also U1.2 (A0); no longer U117.2 (A0)
- net IO_0061: now also U1.1 (E), U1.15 (E); no longer U117.1 (E)
- net NMI_EN: now also RN3.2 (R1), U2.16 (B2)
- net PORT_0X61_EN: now also U1.4 (O0); no longer U117.4 (O0)
- net SPK_EN: now also U2.12 (B6)
- net SPK_GO: now also U2.11 (B7)
- net PORT_61_2: now reaches U15.14 (Q5)
- net PORT_61_2: now also U2.13 (B5)
- net PORT_61_3: now reaches U15.15 (Q4)
- net PORT_61_3: now also U2.14 (B4)
- net PORT_61_4: now reaches U15.16 (Q3)
- net PORT_61_4: now also U2.15 (B3)
- net PORT_61_6: now reaches U15.18 (Q1)
- net PORT_61_6: now also U2.17 (B1)
- net PORT_61_7: now reaches U15.19 (Q0)
- net PORT_61_7: now also U2.18 (B0)
- net IRQ6_JMP: no longer names the net of U16.12
- new net PORT_61_RD: U1.12 (O0), U2.19 (CE)
Other:
- moved on the sheet: U117A, U117B, U117C, U15, U17B
