File: Kicad/640K ISA/640k.kicad_pcb (KiCad board)
At the start: 2 copper layers, 104 x 73.9 mm, 17 parts, among them J9 Bus_ISA_8bit, U1 62256, U2 28C256, U3 AS6C4008, U4 74LS139, U5 74LS138, U6 AS6C1008

Commit message: Updated 640k Gerber files
Parts:
- moved U3 20.3 mm to (147.8, 73.9)
- moved U6 20.3 mm to (127.5, 73.9)
Routing:
- net /A17: track 139.8 -> 109.5 mm, vias 4 -> 5
- net /128K_CS: track 31.5 -> 52.4 mm
- net /512K_CS: track 47.3 -> 26.8 mm
- net /A18: track 161.5 -> 144.7 mm, vias 6 -> 7
- net /D0: track 107.2 -> 91.9 mm
- net /A19: track 106.7 -> 91.4 mm
- net /GND: track 363.1 -> 349.1 mm
- net /D1: track 99.5 -> 88.1 mm
- net /A11: track 113.7 -> 102.2 mm
- net /A16: track 134.9 -> 127.3 mm
- net /D7: track 99.7 -> 92.1 mm
- net /D6: track 97.2 -> 89.5 mm
- net /D5: track 94.6 -> 87.0 mm
- net /D4: track 92.1 -> 84.5 mm
- net /A9: track 112.6 -> 105.0 mm
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
Commit message: 640k update
Parts:
- moved C6 30.2 mm to (174.3, 96.0)
- moved C5 25.4 mm to (174.3, 70.6)
- moved C2 20.9 mm to (117.4, 75.7)
- moved C3 20.9 mm to (137.7, 70.6)
- moved C4 16.3 mm to (158.1, 70.6)
- renumbered U2 to U1, U1 to U2, U6 to U3, U3 to U4, U4 to U5, U5 to U6
