File: Kicad/640K ISA/640k.sch (KiCad schematic (older format))
At the start: 13 parts, among them J9 Bus_ISA_8bit, U1 62256, U2 28C256, U3 AS6C4008, U4 74LS139, U5 74LS138, U6 AS6C1008

Commit message: 640k update
Parts:
- renumbered U2 to U1, U1 to U2, U6 to U3, U3 to U4, U4 to U5, U5 to U6
Other:
- moved on the sheet: C3, C4, C5, C6, U3, U4
