File: Kicad/DMA ISA/DMA.sch (KiCad schematic (older format))
At the start: 14 parts, among them J1 Conn_02x08_Counter_Clockwise, J9 Bus_ISA_8bit, U1 74LS04, U2 74LS573, U3 74LS670, U4 8237, U5 74LS139

Commit message: Update to DMA card
Parts:
- added R3: 27 ohm, Resistor_THT:R_Axial_DIN0207_L6.3mm_D2.5mm_P10.16mm_Horizontal, symbol Device:R
Connections:
- net CLK88: now also R3.2; no longer U1.1
- net CLK88_1: now also R3.1; no longer U1.2
Changed lines of the file:
@@
 Text Label 4625 5400 2    50   ~ 0
 IO_000X
-Text Label 2250 5575 2    50   ~ 0
+Text Label 3875 4875 2    50   ~ 0
 CLK88
-Text Label 2850 5575 0    50   ~ 0
+Text Label 3875 5175 0    50   ~ 0
 CLK88_1
 Text Label 4625 5600 2    50   ~ 0
@@
 Text Label 3800 6050 2    50   ~ 0
 DRQ0_
+$Comp
+L Device:R R3
+U 1 1 623CE352
+P 3875 5025
+F 0 "R3" H 3945 5071 50  0000 L CNN
+F 1 "27 ohm" H 3945 4980 50  0000 L CNN
+F 2 "Resistor_THT:R_Axial_DIN0207_L6.3mm_D2.5mm_P10.16mm_Horizontal" V 3805 5025 50  0001 C CNN
+F 3 "~" H 3875 5025 50  0001 C CNN
+	1    3875 5025
+	-1   0    0    1
+$EndComp
 $EndSCHEMATC

Commit message: DMA update
Parts:
- U3: renamed from U1; footprint (none) -> Package_DIP:DIP-14_W7.62mm
- U4: renamed from U3; value 74LS670 -> 74LS04; footprint Package_DIP:DIP-16_W7.62mm -> Package_DIP:DIP-14_W7.62mm
- U5: renamed from U2; value 74LS573 -> 74LS139; footprint Package_DIP:DIP-20_W7.62mm -> Package_DIP:DIP-16_W7.62mm
- renumbered U4 to U1, U5 to U2, U1 to U3
Changed lines of the file:
@@
 $EndComp
 $Comp
-L 74xx:74LS670 U3
+L 74xx:74LS670 U4
 U 1 1 610632BC
 P 10425 6350
-F 0 "U3" H 10425 7331 50  0000 C CNN
-F 1 "74LS670" H 10425 7240 50  0000 C CNN
-F 2 "Package_DIP:DIP-16_W7.62mm" H 10425 6350 50  0001 C CNN
-F 3 "" H 10425 6350 50  0001 C CNN
+F 0 "U4" H 10425 7331 50  0000 C CNN
+F 1 "74LS04" H 10425 7240 50  0000 C CNN
+F 2 "Package_DIP:DIP-14_W7.62mm" H 10425 6350 50  0001 C CNN
+F 3 "http://www.ti.com/lit/gpn/sn74LS04" H 10425 6350 50  0001 C CNN
 	1    10425 6350
 	1    0    0    -1
@@
 5+
 $Comp
-L Interface:8237 U4
+L Interface:8237 U1
 U 1 1 61463853
 P 5325 6200
-F 0 "U4" H 5325 4511 50  0000 C CNN
+F 0 "U1" H 5325 4511 50  0000 C CNN
 F 1 "8237" H 5325 4420 50  0000 C CNN
 F 2 "Package_DIP:DIP-40_W15.24mm" H 5325 6400 50  0001 C CNN
@@
 CLK88_1
 $Comp
-L 74xx:74LS04 U1
+L 74xx:74LS04 U3
 U 1 1 61470FF9
 P 2550 5575
-F 0 "U1" H 2550 5892 50  0000 C CNN
+F 0 "U3" H 2550 5892 50  0000 C CNN
 F 1 "74LS04" H 2550 5801 50  0000 C CNN
 F 2 "Package_DIP:DIP-14_W7.62mm" H 2550 5575 50  0001 C CNN
@@
 $EndComp
 $Comp
-L 74xx:74LS04 U1
+L 74xx:74LS04 U3
 U 7 1 61471E02
 P 2450 7200
-F 0 "U1" V 2083 7200 50  0000 C CNN
+F 0 "U3" V 2083 7200 50  0000 C CNN
 F 1 "74LS04" V 2174 7200 50  0000 C CNN
 F 2 "Package_DIP:DIP-14_W7.62mm" H 2450 7200 50  0001 C CNN
@@
 $EndComp
 $Comp
-L 74xx:74LS04 U1
+L 74xx:74LS04 U3
 U 2 1 61472C9C
 P 2475 6125
-F 0 "U1" H 2475 6442 50  0000 C CNN
+F 0 "U3" H 2475 6442 50  0000 C CNN
 F 1 "74LS04" H 2475 6351 50  0000 C CNN
 F 2 "Package_DIP:DIP-14_W7.62mm" H 2475 6125 50  0001 C CNN
@@
 A15
 $Comp
-L 74xx:74LS573 U2
+L 74xx:74LS573 U5
 U 1 1 610661C4
 P 10450 9225
-F 0 "U2" H 10450 10206 50  0000 C CNN
-F 1 "74LS573" H 10450 10115 50  0000 C CNN
-F 2 "Package_DIP:DIP-20_W7.62mm" H 10450 9225 50  0001 C CNN
-F 3 "74xx/74hc573.pdf" H 10450 9225 50  0001 C CNN
+F 0 "U5" H 10450 10206 50  0000 C CNN
+F 1 "74LS139" H 10450 10115 50  0000 C CNN
+F 2 "Package_DIP:DIP-16_W7.62mm" H 10450 9225 50  0001 C CNN
+F 3 "http://www.ti.com/lit/ds/symlink/sn74ls139a.pdf" H 10450 9225 50  0001 C CNN
 	1    10450 9225
 	1    0    0    -1
@@
 AEN_OE
 $Comp
-L 74xx:74LS139 U5
+L 74xx:74LS139 U2
 U 1 1 61463DE3
 P 10375 3175
-F 0 "U5" H 10375 3542 50  0000 C CNN
+F 0 "U2" H 10375 3542 50  0000 C CNN
 F 1 "74LS139" H 10375 3451 50  0000 C CNN
 F 2 "Package_DIP:DIP-16_W7.62mm" H 10375 3175 50  0001 C CNN
@@
 $EndComp
 $Comp
-L 74xx:74LS139 U5
+L 74xx:74LS139 U2
 U 3 1 61464882
 P 10350 4175
-F 0 "U5" V 9983 4175 50  0000 C CNN
+F 0 "U2" V 9983 4175 50  0000 C CNN
 F 1 "74LS139" V 10074 4175 50  0000 C CNN
 F 2 "Package_DIP:DIP-16_W7.62mm" H 10350 4175 50  0001 C CNN
@@
 760_EN
 $Comp
-L 74xx:74LS04 U1
+L 74xx:74LS04 U3
 U 3 1 614D3A02
 P 2475 6625
-F 0 "U1" H 2475 6942 50  0000 C CNN
+F 0 "U3" H 2475 6942 50  0000 C CNN
 F 1 "74LS04" H 2475 6851 50  0000 C CNN
-F 2 "" H 2475 6625 50  0001 C CNN
+F 2 "Package_DIP:DIP-14_W7.62mm" H 2475 6625 50  0001 C CNN
 F 3 "http://www.ti.com/lit/gpn/sn74LS04" H 2475 6625 50  0001 C CNN
 	3    2475 6625

Commit message: Gerber update
Parts:
- U4: value 74LS04 -> 74LS670; footprint Package_DIP:DIP-14_W7.62mm -> Package_DIP:DIP-16_W7.62mm
- U5: value 74LS139 -> 74LS573; footprint Package_DIP:DIP-16_W7.62mm -> Package_DIP:DIP-20_W7.62mm
- renumbered C8 to C5
Changed lines of the file:
@@
 P 10425 6350
 F 0 "U4" H 10425 7331 50  0000 C CNN
-F 1 "74LS04" H 10425 7240 50  0000 C CNN
-F 2 "Package_DIP:DIP-14_W7.62mm" H 10425 6350 50  0001 C CNN
+F 1 "74LS670" H 10425 7240 50  0000 C CNN
+F 2 "Package_DIP:DIP-16_W7.62mm" H 10425 6350 50  0001 C CNN
 F 3 "http://www.ti.com/lit/gpn/sn74LS04" H 10425 6350 50  0001 C CNN
 	1    10425 6350
@@
 Text Label 4625 4900 2    50   ~ 0
 A0
-Text Label 10450 8425 0    50   ~ 0
-5+
 Text Label 10450 10025 0    50   ~ 0
 GND
@@
 GND
 $Comp
-L pspice:CAP C8
+L pspice:CAP C5
 U 1 1 61169660
 P 2900 5025
-F 0 "C8" V 2585 5025 50  0000 C CNN
+F 0 "C5" V 2585 5025 50  0000 C CNN
 F 1 "0.1uF" V 2676 5025 50  0000 C CNN
 F 2 "Capacitor_THT:C_Disc_D4.3mm_W1.9mm_P5.00mm" H 2900 5025 50  0001 C CNN
@@
 Text Label 10950 8925 0    50   ~ 0
 A13
-Text Label 10950 8825 0    50   ~ 0
-A14
-Text Label 10950 8725 0    50   ~ 0
-A15
-$Comp
-L 74xx:74LS573 U5
-U 1 1 610661C4
-P 10450 9225
-F 0 "U5" H 10450 10206 50  0000 C CNN
-F 1 "74LS139" H 10450 10115 50  0000 C CNN
-F 2 "Package_DIP:DIP-16_W7.62mm" H 10450 9225 50  0001 C CNN
-F 3 "http://www.ti.com/lit/ds/symlink/sn74ls139a.pdf" H 10450 9225 50  0001 C CNN
-	1    10450 9225
-	1    0    0    -1
-$EndComp
 Text Label 10950 9225 0    50   ~ 0
 A10
@@
 	-1   0    0    1
 $EndComp
+$Comp
+L 74xx:74LS573 U5
+U 1 1 610661C4
+P 10450 9225
+F 0 "U5" H 10450 10206 50  0000 C CNN
+F 1 "74LS573" H 10450 10115 50  0000 C CNN
+F 2 "Package_DIP:DIP-20_W7.62mm" H 10450 9225 50  0001 C CNN
+F 3 "http://www.ti.com/lit/ds/symlink/sn74ls139a.pdf" H 10450 9225 50  0001 C CNN
+	1    10450 9225
+	1    0    0    -1
+$EndComp
+Text Label 10950 8725 0    50   ~ 0
+A15
+Text Label 10950 8825 0    50   ~ 0
+A14
+Text Label 10450 8425 0    50   ~ 0
+5+
 $EndSCHEMATC

Commit message: Updated DMA card
Parts:
- renumbered R2 to R1, R1 to R2
Other:
- moved on the sheet: C4
Changed lines of the file:
@@
 	0    1    1    0
 $EndComp
-Text Label 5650 3875 0    50   ~ 0
-GND
-Text Label 5150 3875 2    50   ~ 0
+Text Label 6225 4200 0    50   ~ 0
+GND
+Text Label 5725 4200 2    50   ~ 0
 5+
 $Comp
 L pspice:CAP C4
 U 1 1 6106BA7C
-P 5400 3875
-F 0 "C4" V 5085 3875 50  0000 C CNN
-F 1 "0.1uF" V 5176 3875 50  0000 C CNN
-F 2 "Capacitor_THT:C_Disc_D4.3mm_W1.9mm_P5.00mm" H 5400 3875 50  0001 C CNN
-F 3 "~" H 5400 3875 50  0001 C CNN
-	1    5400 3875
+P 5975 4200
+F 0 "C4" V 5660 4200 50  0000 C CNN
+F 1 "0.1uF" V 5751 4200 50  0000 C CNN
+F 2 "Capacitor_THT:C_Disc_D4.3mm_W1.9mm_P5.00mm" H 5975 4200 50  0001 C CNN
+F 3 "~" H 5975 4200 50  0001 C CNN
+	1    5975 4200
 	0    1    1    0
 $EndComp
@@
 EOP
 $Comp
-L Device:R R1
+L Device:R R2
 U 1 1 6146BFF5
 P 6950 6250
-F 0 "R1" H 7020 6296 50  0000 L CNN
+F 0 "R2" H 7020 6296 50  0000 L CNN
 F 1 "10k ohm" H 7020 6205 50  0000 L CNN
 F 2 "Resistor_THT:R_Axial_DIN0207_L6.3mm_D2.5mm_P10.16mm_Horizontal" V 6880 6250 50  0001 C CNN
@@
 REFRQ
 $Comp
-L Device:R R2
+L Device:R R1
 U 1 1 6174F842
 P 3800 6200
-F 0 "R2" H 3870 6246 50  0000 L CNN
+F 0 "R1" H 3870 6246 50  0000 L CNN
 F 1 "10k ohm" H 3870 6155 50  0000 L CNN
 F 2 "Resistor_THT:R_Axial_DIN0207_L6.3mm_D2.5mm_P10.16mm_Horizontal" V 3730 6200 50  0001 C CNN
