File: Kicad/Multi ATX 7 ISA/Multi.kicad_pcb (KiCad board)
At the start: 2 copper layers, 182.9 x 172.7 mm, 107 parts, among them J1 Bus_ISA_8bit, J10 Conn_02x08_Counter_Clockwise, J11 Conn_02x08_Counter_Clockwise, J12 Bus_ISA_8bit, J13 Bus_ISA_8bit, J14 Bus_ISA_8bit, J2 Mini-DIN-6, J3 SPK, J6 PWR ON, J7 Bus_ISA_8bit, J8 Bus_ISA_8bit, J9 Bus_ISA_8bit, SW1 RESET, U1 74LS139, U11 8284, U117 74LS139, U12 74LS138, U13 74LS138, U14 74LS74, U15 74LS573, U16 74LS04, U17 74LS139, U19 82C42/83C42, U2 74LS245, U20 74LS07, U3 33 ohm, U9 74LS138, Y2 14.31818 MHz

Commit message: fixed 5+ pin on PCB
Connections:
- U1 pad 16: Net-(U1-Pad16) -> /5+
Routing:
- net /5+: track 1118.6 -> 1121.9 mm

Commit message: Updated Kicad files
Other:
- board text added: "EMM COMPUTERS 8-BIT MAIN BOARD Copyright (C) 2022 EMM www.homebrew8088.com"
- board text removed: "EMM COMPUTERS 8-BIT MAIN BOARD Copyright (C) 2021 EMM www.homebrew8088.com"
Changed lines of the file:
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@@
   (gr_line (start 141.986 18.542) (end 141.986 191.262) (layer Edge.Cuts) (width 0.05))
   (gr_line (start -40.894 18.542) (end -40.894 191.262) (layer Edge.Cuts) (width 0.05))
-  (gr_text "EMM COMPUTERS\n8-BIT MAIN BOARD\nCopyright (C) 2021 EMM\nwww.homebrew8088.com\n" (at -18.796 24.892) (layer F.SilkS)
+  (gr_text "EMM COMPUTERS\n8-BIT MAIN BOARD\nCopyright (C) 2022 EMM\nwww.homebrew8088.com\n" (at -18.796 24.892) (layer F.SilkS)
     (effects (font (size 1.5 1.5) (thickness 0.3)) (justify left))
   )

Commit message: Update main board
Parts:
- removed the ? at (148.6, 46.2)
- renumbered U3 to R112, U15 to U1, U14 to U10, U117 to U11, U17 to U12, U1 to U13, U19 to U3, U20 to U4, U13 to U5, U16 to U6, U9 to U7, U12 to U8, U11 to U9
