File: Kicad/Multi ATX 7 ISA/Multi.sch (KiCad schematic (older format))
At the start: 76 parts, among them J1 Bus_ISA_8bit, J10 Conn_02x08_Counter_Clockwise, J11 Conn_02x08_Counter_Clockwise, J12 Bus_ISA_8bit, J13 Bus_ISA_8bit, J14 Bus_ISA_8bit, J2 Mini-DIN-6, J3 SPK, J6 PWR ON, J7 Bus_ISA_8bit, J8 Bus_ISA_8bit, J9 Bus_ISA_8bit, SW1 RESET, U1 74LS139, U11 8284, U117 74LS139, U12 74LS138, U13 74LS138, U14 74LS74, U15 74LS573, U16 74LS04, U17 74LS139, U19 82C42/83C42, U2 74LS245, U20 74LS07, U3 33 ohm, U9 74LS138, Y2 14.31818 MHz

Commit message: fixed 5+ pin on PCB
Connections:
- net 5+: now also U1.16 (VCC)
Changed lines of the file:
@@
 	1    0    0    -1
 $EndComp
+Text Label 9850 13950 0    50   ~ 0
+5+
 $EndSCHEMATC

Commit message: Update main board
Parts:
- renumbered U3 to R112, U15 to U1, U14 to U10, U117 to U11, U17 to U12, U1 to U13, U19 to U3, U20 to U4, U13 to U5, U16 to U6, U9 to U7, U12 to U8, U11 to U9
Changed lines of the file:
@@
 $EndDescr
 $Comp
-L 74xx:74LS139 U117
+L 74xx:74LS139 U11
 U 2 1 5FEFF66E
 P 5300 13400
-F 0 "U117" H 5300 13767 50  0000 C CNN
+F 0 "U11" H 5300 13767 50  0000 C CNN
 F 1 "74LS139" H 5300 13676 50  0000 C CNN
 F 2 "Package_DIP:DIP-16_W7.62mm" H 5300 13400 50  0001 C CNN
@@
 GND
 $Comp
-L 74xx:74LS74 U14
+L 74xx:74LS74 U10
 U 1 1 5FF31A0C
 P 6650 7125
-F 0 "U14" H 6650 7606 50  0001 C CNN
+F 0 "U10" H 6650 7606 50  0000 C CNN
 F 1 "74LS74" H 6650 7514 50  0000 C CNN
 F 2 "Package_DIP:DIP-14_W7.62mm" H 6650 7125 50  0001 C CNN
@@
 $EndComp
 $Comp
-L 74xx:74LS74 U14
+L 74xx:74LS74 U10
 U 2 1 5FF327F5
 P 6650 7825
-F 0 "U14" H 6650 8306 50  0001 C CNN
+F 0 "U10" H 6650 8306 50  0000 C CNN
 F 1 "74LS74" H 6650 8214 50  0000 C CNN
 F 2 "Package_DIP:DIP-14_W7.62mm" H 6650 7825 50  0001 C CNN
@@
 $EndComp
 $Comp
-L 74xx:74LS74 U14
+L 74xx:74LS74 U10
 U 3 1 5FF335DC
 P 6650 8575
-F 0 "U14" H 6880 8621 50  0001 L CNN
+F 0 "U10" H 6880 8621 50  0000 L CNN
 F 1 "74LS74" V 6375 8575 50  0000 C CNN
 F 2 "Package_DIP:DIP-14_W7.62mm" H 6650 8575 50  0001 C CNN
@@
 SPK_PIN
 $Comp
-L 74xx:74LS138 U13
+L 74xx:74LS138 U5
 U 1 1 5FF39086
 P 3150 13650
-F 0 "U13" H 3150 14431 50  0001 C CNN
+F 0 "U5" H 3150 14431 50  0000 C CNN
 F 1 "74LS138" H 3150 14339 50  0000 C CNN
 F 2 "Package_DIP:DIP-16_W7.62mm" H 3150 13650 50  0001 C CNN
@@
 5+
 $Comp
-L Device:R U3
+L Device:R R112
 U 1 1 5FF4B88D
 P 5150 11550
-F 0 "U3" H 5220 11596 50  0001 L CNN
+F 0 "R112" H 5220 11596 50  0001 L CNN
 F 1 "33 ohm" V 5035 11550 50  0000 C CNN
 F 2 "Resistor_THT:R_Axial_DIN0207_L6.3mm_D2.5mm_P10.16mm_Horizontal" V 5080 11550 50  0001 C CNN
@@
 5+
 $Comp
-L 74xx:74LS04 U16
+L 74xx:74LS04 U6
 U 1 1 5FF518D3
 P 10250 6050
-F 0 "U16" H 10250 6367 50  0001 C CNN
+F 0 "U6" H 10250 6367 50  0000 C CNN
 F 1 "74LS04" H 10250 6275 50  0000 C CNN
 F 2 "Package_DIP:DIP-14_W7.62mm" H 10250 6050 50  0001 C CNN
@@
 $EndComp
 $Comp
-L 74xx:74LS04 U16
+L 74xx:74LS04 U6
 U 2 1 5FF5211D
 P 10250 6375
-F 0 "U16" H 10250 6692 50  0001 C CNN
+F 0 "U6" H 10250 6692 50  0000 C CNN
 F 1 "74LS04" H 10250 6600 50  0000 C CNN
 F 2 "Package_DIP:DIP-14_W7.62mm" H 10250 6375 50  0001 C CNN
@@
 $EndComp
 $Comp
-L 74xx:74LS04 U16
+L 74xx:74LS04 U6
 U 3 1 5FF5313C
 P 10250 6700
-F 0 "U16" H 10250 7017 50  0001 C CNN
+F 0 "U6" H 10250 7017 50  0001 C CNN
 F 1 "74LS04" H 10250 6925 50  0000 C CNN
 F 2 "Package_DIP:DIP-14_W7.62mm" H 10250 6700 50  0001 C CNN
@@
 $EndComp
 $Comp
-L 74xx:74LS04 U16
+L 74xx:74LS04 U6
 U 7 1 5FF55544
 P 10175 8075
-F 0 "U16" V 9808 8075 50  0001 C CNN
+F 0 "U6" V 9808 8075 50  0000 C CNN
 F 1 "74LS04" V 9900 8075 50  0000 C CNN
 F 2 "Package_DIP:DIP-14_W7.62mm" H 10175 8075 50  0001 C CNN
@@
 NMI_EN_139
 $Comp
-L 74xx:74LS139 U17
+L 74xx:74LS139 U12
 U 1 1 5FF5A2F8
 P 7475 12825
-F 0 "U17" H 7475 13192 50  0001 C CNN
+F 0 "U12" H 7475 13192 50  0000 C CNN
 F 1 "74LS139" H 7475 13100 50  0000 C CNN
 F 2 "Package_DIP:DIP-16_W7.62mm" H 7475 12825 50  0001 C CNN
@@
 $EndComp
 $Comp
-L 74xx:74LS139 U17
+L 74xx:74LS139 U12
 U 3 1 5FF5AFDE
 P 7425 14075
-F 0 "U17" V 7058 14075 50  0001 C CNN
+F 0 "U12" V 7058 14075 50  0000 C CNN
 F 1 "74LS139" V 7150 14075 50  0000 C CNN
 F 2 "Package_DIP:DIP-16_W7.62mm" H 7425 14075 50  0001 C CNN
@@
 CH_CK
 $Comp
-L 74xx:74LS573 U15
+L 74xx:74LS573 U1
 U 1 1 60133ADF
 P 13250 13375
-F 0 "U15" H 13250 14356 50  0000 C CNN
+F 0 "U1" H 13250 14356 50  0000 C CNN
 F 1 "74LS573" H 13250 14265 50  0000 C CNN
 F 2 "Package_DIP:DIP-20_W7.62mm" H 13250 13375 50  0001 C CNN
@@
 IO_0061
 $Comp
-L 74xx:74LS139 U117
+L 74xx:74LS139 U11
 U 1 1 60244EB2
 P 5300 12800
-F 0 "U117" H 5300 13167 50  0000 C CNN
+F 0 "U11" H 5300 13167 50  0000 C CNN
 F 1 "74LS139" H 5300 13076 50  0000 C CNN
 F 2 "Package_DIP:DIP-16_W7.62mm" H 5300 12800 50  0001 C CNN
@@
 $EndComp
 $Comp
-L 74xx:74LS139 U117
+L 74xx:74LS139 U11
 U 3 1 60245F47
 P 5300 14075
-F 0 "U117" V 4933 14075 50  0000 C CNN
+F 0 "U11" V 4933 14075 50  0000 C CNN
 F 1 "74LS139" V 5024 14075 50  0000 C CNN
 F 2 "Package_DIP:DIP-16_W7.62mm" H 5300 14075 50  0001 C CNN
@@
 CH_CK
 $Comp
-L W83C42P:W83C42P U19
+L W83C42P:W83C42P U3
 U 1 1 60848F25
 P 9050 8875
-F 0 "U19" H 9050 8940 50  0000 C CNN
+F 0 "U3" H 9050 8940 50  0000 C CNN
 F 1 "82C42/83C42" H 9050 8849 50  0000 C CNN
 F 2 "Package_LCC:PLCC-44_THT-Socket" H 9050 8875 50  0001 C CNN
@@
 5+
 $Comp
-L 74xx:74LS138 U12
+L 74xx:74LS138 U8
 U 1 1 5FF38345
 P 1600 13625
-F 0 "U12" H 1600 14406 50  0001 C CNN
+F 0 "U8" H 1600 14406 50  0000 C CNN
 F 1 "74LS138" H 1600 14314 50  0000 C CNN
 F 2 "Package_DIP:DIP-16_W7.62mm" H 1600 13625 50  0001 C CNN
@@
 $EndComp
 $Comp
-L 74xx:74LS138 U9
+L 74xx:74LS138 U7
 U 1 1 5FF377FE
 P 1650 11950
-F 0 "U9" H 1650 12731 50  0001 C CNN
+F 0 "U7" H 1650 12731 50  0000 C CNN
 F 1 "74LS138" H 1650 12639 50  0000 C CNN
 F 2 "Package_DIP:DIP-16_W7.62mm" H 1650 11950 50  0001 C CNN
@@
 $EndComp
 $Comp
-L 74xx:74LS139 U17
+L 74xx:74LS139 U12
 U 2 1 60138DE8
 P 7475 13425
-F 0 "U17" H 7475 13792 50  0000 C CNN
+F 0 "U12" H 7475 13792 50  0000 C CNN
 F 1 "74LS139" H 7475 13701 50  0000 C CNN
 F 2 "Package_DIP:DIP-16_W7.62mm" H 7475 13425 50  0001 C CNN
@@
 $EndComp
 $Comp
-L 74xx:74LS07 U20
+L 74xx:74LS07 U4
 U 1 1 6088A1DA
 P 11825 9250
-F 0 "U20" H 11825 9567 50  0000 C CNN
+F 0 "U4" H 11825 9567 50  0000 C CNN
 F 1 "74LS07" H 11825 9476 50  0000 C CNN
 F 2 "Package_DIP:DIP-14_W7.62mm" H 11825 9250 50  0001 C CNN
@@
 $EndComp
 $Comp
-L 74xx:74LS07 U20
+L 74xx:74LS07 U4
 U 2 1 6088AC3C
 P 11475 9725
-F 0 "U20" H 11475 10042 50  0000 C CNN
+F 0 "U4" H 11475 10042 50  0000 C CNN
 F 1 "74LS07" H 11475 9951 50  0000 C CNN
 F 2 "Package_DIP:DIP-14_W7.62mm" H 11475 9725 50  0001 C CNN
@@
 $EndComp
 $Comp
-L 74xx:74LS07 U20
+L 74xx:74LS07 U4
 U 7 1 6088CF4D
 P 11675 10350
-F 0 "U20" V 11308 10350 50  0000 C CNN
+F 0 "U4" V 11308 10350 50  0000 C CNN
 F 1 "74LS07" V 11399 10350 50  0000 C CNN
 F 2 "Package_DIP:DIP-14_W7.62mm" H 11675 10350 50  0001 C CNN
@@
 KBD_CLK_INVERTED
 $Comp
-L 74xx:74LS04 U16
+L 74xx:74LS04 U6
 U 5 1 60896907
 P 10250 7025
-F 0 "U16" H 10250 7342 50  0000 C CNN
+F 0 "U6" H 10250 7342 50  0000 C CNN
 F 1 "74LS04" H 10250 7251 50  0000 C CNN
 F 2 "Package_DIP:DIP-14_W7.62mm" H 10250 7025 50  0001 C CNN
@@
 $EndComp
 $Comp
-L Timer:8284 U11
+L Timer:8284 U9
 U 1 1 5FF2451F
 P 4300 7700
-F 0 "U11" H 4300 8781 50  0000 C CNN
+F 0 "U9" H 4300 8781 50  0000 C CNN
 F 1 "8284" H 4300 8690 50  0000 C CNN
 F 2 "Package_DIP:DIP-18_W7.62mm" H 4300 7700 50  0001 C CIN
@@
 $EndComp
 $Comp
-L 74xx:74LS139 U1
+L 74xx:74LS139 U13
 U 1 1 61B29026
 P 9350 12950
-F 0 "U1" H 9350 13317 50  0000 C CNN
+F 0 "U13" H 9350 13317 50  0000 C CNN
 F 1 "74LS139" H 9350 13226 50  0000 C CNN
 F 2 "Package_DIP:DIP-16_W7.62mm" H 9350 12950 50  0001 C CNN
@@
 $EndComp
 $Comp
-L 74xx:74LS139 U1
+L 74xx:74LS139 U13
 U 2 1 61B2A28C
 P 9350 13450
-F 0 "U1" H 9350 13817 50  0000 C CNN
+F 0 "U13" H 9350 13817 50  0000 C CNN
 F 1 "74LS139" H 9350 13726 50  0000 C CNN
 F 2 "Package_DIP:DIP-16_W7.62mm" H 9350 13450 50  0001 C CNN
@@
 $EndComp
 $Comp
-L 74xx:74LS139 U1
+L 74xx:74LS139 U13
 U 3 1 61B2BC61
 P 9350 13950
-F 0 "U1" V 8983 13950 50  0000 C CNN
+F 0 "U13" V 8983 13950 50  0000 C CNN
 F 1 "74LS139" V 9074 13950 50  0000 C CNN
 F 2 "Package_DIP:DIP-16_W7.62mm" H 9350 13950 50  0001 C CNN
@@
 5+
 $Comp
-L 74xx:74LS04 U16
+L 74xx:74LS04 U6
 U 6 1 6028B501
 P 10250 7675
-F 0 "U16" H 10250 7992 50  0001 C CNN
+F 0 "U6" H 10250 7992 50  0001 C CNN
 F 1 "74LS04" H 10250 7900 50  0000 C CNN
 F 2 "Package_DIP:DIP-14_W7.62mm" H 10250 7675 50  0001 C CNN
@@
 $EndComp
 $Comp
-L 74xx:74LS04 U16
+L 74xx:74LS04 U6
 U 4 1 602C2470
 P 10250 7350
-F 0 "U16" H 10250 7667 50  0000 C CNN
+F 0 "U6" H 10250 7667 50  0000 C CNN
 F 1 "74LS04" H 10250 7576 50  0000 C CNN
 F 2 "Package_DIP:DIP-14_W7.62mm" H 10250 7350 50  0001 C CNN
