File: Kicad/Multi ATX 10 ISA/Multi.kicad_pcb (KiCad board)
At the start: 2 copper layers, 182.9 x 172.7 mm, 106 parts, among them J1 Bus_ISA_8bit, J10 Conn_02x08_Counter_Clockwise, J11 Conn_02x08_Counter_Clockwise, J12 Bus_ISA_8bit, J13 Bus_ISA_8bit, J14 Bus_ISA_8bit, J2 Mini-DIN-6, J3 SPK, J6 PWR ON, J7 Bus_ISA_8bit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

Commit message: Added 10 Slot main board
Parts:
- removed the REF** at (-26.9, 183.6)
- removed the REF** at (-26.9, 28.7)
- added C20: 0.1uF, Capacitor_THT:C_Disc_D4.3mm_W1.9mm_P5.00mm, F.Cu at (-63.0, 44.7)
- added C21: 0.1uF, Capacitor_THT:C_Disc_D4.3mm_W1.9mm_P5.00mm, F.Cu at (-63.0, 120.6)
- added C30: 0.1uF, Capacitor_THT:C_Disc_D4.3mm_W1.9mm_P5.00mm, F.Cu at (-22.4, 44.7)
- added C31: 0.1uF, Capacitor_THT:C_Disc_D4.3mm_W1.9mm_P5.00mm, F.Cu at (-42.7, 120.6)
- added C32: 0.1uF, Capacitor_THT:C_Disc_D4.3mm_W1.9mm_P5.00mm, F.Cu at (-22.4, 120.6)
- added C33: 0.1uF, Capacitor_THT:C_Disc_D4.3mm_W1.9mm_P5.00mm, F.Cu at (-42.7, 44.7)
- added J15: Bus_ISA_8bit, Motherboard:8-bit-ISA, F.Cu at (21.3, 43.9)
- added J4: Bus_ISA_8bit, Motherboard:8-bit-ISA, F.Cu at (-19.3, 43.9)
- added J5: Bus_ISA_8bit, Motherboard:8-bit-ISA, F.Cu at (1.02, 43.9)
- added R: L, Motherboard:Large_Via, F.Cu at (-97.3, 37.8)
- added R: L, Motherboard:Large_Via, F.Cu at (-98.8, 40.4)
- added R: L, Motherboard:Large_Via, F.Cu at (-77.0, 37.8)
- added R: L, Motherboard:Large_Via, F.Cu at (-78.5, 40.4)
- added R: L, Motherboard:Large_Via, F.Cu at (-56.6, 37.8)
- added R: L, Motherboard:Large_Via, F.Cu at (-58.2, 40.4)
- added REF**: MountingHole_3.7mm, MountingHole:MountingHole_3.7mm, F.Cu at (-87.9, 183.6)
- added REF**: MountingHole_3.7mm, MountingHole:MountingHole_3.7mm, F.Cu at (-87.9, 28.7)
- moved C24 61.0 mm to (-92.5, 44.7)
- moved C27 61.0 mm to (-92.5, 120.6)
- moved J1 61.0 mm to (-39.6, 43.9)
- moved J12 61.0 mm to (-100.6, 43.9)
- moved J14 61.0 mm to (-59.9, 43.9)
- moved REF** 61.0 mm to (36.6, 183.6)
- moved REF** 61.0 mm to (-9.14, 183.6)
- moved REF** 61.0 mm to (36.6, 28.7)
- moved REF** 61.0 mm to (-9.14, 28.7)
- moved C11 61.0 mm to (-83.3, 120.6)
- moved C15 61.0 mm to (-83.3, 44.7)
- moved J13 61.0 mm to (-80.3, 43.9)
- moved RN1 21.6 mm to (8.13, 32.0)
Routing:
- net /GND: track 1377.2 -> 1567.9 mm
- net /12+: track 452.9 -> 600.3 mm
- net /5+: track 1121.9 -> 1261.8 mm
- net /12-: track 422.7 -> 546.5 mm
- net /D4: track 207.8 -> 271.9 mm
- net /DACK3: track 182.1 -> 246.2 mm
- net /5-: track 128.2 -> 192.3 mm
- net /RESOUT: track 259.1 -> 323.2 mm
- net /IRQ2: track 128.2 -> 192.3 mm
- net /DRQ2: track 153.9 -> 218.0 mm
- net /DACK2: track 209.8 -> 273.9 mm
- net /D1: track 199.4 -> 263.6 mm
- net /A2: track 268.7 -> 332.9 mm
- net /A17: track 128.2 -> 192.3 mm
- net /A14: track 207.5 -> 271.7 mm
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Other:
- board size 182.9 x 172.7 mm -> 243.8 x 172.7 mm
- board text added: "EMM COMPUTERS 8-BIT MAIN BOARD / 10 SLOT Copyright (C) 2022 EMM www.homebrew8088.com"
- board text removed: "EMM COMPUTERS 8-BIT MAIN BOARD Copyright (C) 2022 EMM www.homebrew8088.com"
