File: Kicad/386EX/386EX.kicad_pcb (KiCad board)
At the start: 2 copper layers, 132 x 73.9 mm, 23 parts, among them J1 Conn_02x08_Counter_Clockwise, J2 Bus_ISA_8bit, J3 Conn_01x02, J4 Conn_01x03, J5 Conn_01x02, J6 Conn_01x03, J7 Conn_01x02, J8 Conn_01x08, U1 I386EX_PQFP, U2 8284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

Commit message: updates to 386
Parts:
- 8_BIT_BUS_EN1: renamed from J7; value Conn_01x02 -> 8 BIT BUS EN
- CLK2_SEL1: renamed from J4; value Conn_01x03 -> CLK2 SEL
- HOLDA_EN1: renamed from J5; value Conn_01x02 -> HOLDA EN
- J8: value Conn_01x08 -> Conn_01x09; footprint Connector_PinHeader_2.54mm:PinHeader_1x08_P2.54mm_Vertical -> Connector_PinHeader_2.54mm:PinHeader_1x09_P2.54mm_Vertical
- OSC_EN1: renamed from J6; value Conn_01x03 -> OSC EN
- READY_PIN_EN1: renamed from J3; value Conn_01x02 -> READY PIN EN
- U1: value I386EX_PQFP -> I386EX
- X1: value CXO_DIP8 -> 33MHz
- moved R1 39.1 mm to (126.5, 73.2), turned to 270 degrees
- moved J8 22.6 mm to (126.5, 97.8), turned to 0 degrees
- moved READY_PIN_EN1 17.3 mm to (135.9, 74.7), turned to 90 degrees
- moved HOLDA_EN1 17.2 mm to (135.9, 85.9), turned to 90 degrees
- moved 8_BIT_BUS_EN1 10.9 mm to (135.9, 80.3), turned to 90 degrees
- moved R3 7.15 mm to (225.3, 88.9)
- moved R7 5.55 mm to (164.1, 72.1)
- moved OSC_EN1 4.83 mm to (243.3, 94.7)
- moved C1 4.20 mm to (158.1, 83.3)
- moved C3 3.54 mm to (217.9, 85.7)
- moved U4 3.54 mm to (212.1, 73.2)
- moved C4 3.54 mm to (215.4, 75.8)
- moved U3 3.54 mm to (214.6, 83.1)
- moved Y1 1.63 mm to (244.9, 80.8)
- moved C2 0.51 mm to (232.0, 75.2)
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Connections:
- R1 pad 3: /HOLDA_JMP -> Net-(R1-Pad3)
- R1 pad 4: Net-(R1-Pad4) -> /8_BIT_EN
- R1 pad 6: Net-(R1-Pad6) -> /HOLDA_JMP
- R1 pad 9: /8_BIT_EN -> Net-(R1-Pad9)
- R7 pad 2: /PU_257 -> /SMIACT
- R7 pad 3: Net-(R7-Pad3) -> /TRST
- R7 pad 4: Net-(R7-Pad4) -> /PIPELINE_EN
- R7 pad 5: /PIPELINE_EN -> Net-(R7-Pad5)
- R7 pad 6: /FLT -> Net-(R7-Pad6)
- R7 pad 7: /SMIACT -> /FLT
- R7 pad 9: /TRST -> /PU_257
- U1 pad 110: /RESET -> /RESET_
- U1 pad 39: Net-(U1-Pad39) -> /BHE
- U3 pad 8: Net-(U3-Pad8) -> /GND
- U4 pad 5: (no net) -> /RESET
- U4 pad 6: (no net) -> /RESET_
Routing:
- net /5+: track 0.00 -> 491.8 mm, vias 0 -> 33
- net /GND: track 0.00 -> 479.8 mm, vias 0 -> 30
- net /RESET: track 0.00 -> 164.6 mm, vias 0 -> 6
- net /HF_PCLK: track 0.00 -> 135.7 mm, vias 0 -> 6
- net /SPK_GO: track 0.00 -> 126.0 mm, vias 0 -> 4
- net /SPK_OUT: track 0.00 -> 124.5 mm, vias 0 -> 4
- net /NMI: track 0.00 -> 121.4 mm, vias 0 -> 3
- net /ALE: track 0.00 -> 118.6 mm, vias 0 -> 4
- net /D7: track 6.11 -> 111.2 mm, vias 1 -> 4
- net /HOLDA: track 0.00 -> 105.0 mm, vias 0 -> 5
- net /HOLDA_JMP: track 0.00 -> 104.7 mm, vias 0 -> 3
- net /D6: track 6.11 -> 109.2 mm, vias 1 -> 4
- net /D5: track 6.11 -> 106.9 mm, vias 1 -> 4
- net /D4: track 6.11 -> 104.6 mm, vias 1 -> 4
- net /D3: track 6.11 -> 103.2 mm, vias 1 -> 4
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Other:
- board text added: "5+"
- board text added: "8284 CLK"
- board text added: "BHE"
- board text added: "CLK2"
- board text added: "D10"
- board text added: "D11"
- board text added: "D12"
- board text added: "D13"
- board text added: "D14"
- board text added: "D15"
- board text added: "D8"
- board text added: "D9"
- board text added: "EN PIN"
- board text added: "GND"
- board text added: "OSC CLK"
