File: Kicad/CH376S Module/CH376S Module.sch (KiCad schematic (older format))
At the start: 14 parts, among them P1 HEADER, U1 CH376, U2 LM1117-3.3, Y2 12 MHz

Commit message: updates to 386
Connections:
- net 5+: no longer C3.1
- net GND: no longer C3.2
Changed lines of the file:
@@
 	1    0    0    -1
 $EndComp
-Text Label 4525 1900 3    50   ~ 0
-GND
 Text Label 4950 1925 3    50   ~ 0
 GND
@@
 Text Label 4950 1725 1    50   ~ 0
 5+
-Text Label 4525 1700 1    50   ~ 0
-5+
 $Comp
