File: Kicad/8088 MAX ISA/8088.kicad_pcb (KiCad board)
At the start: 2 copper layers, 175 x 73.9 mm, 35 parts, among them J1 Conn_02x08_Counter_Clockwise, J9 Bus_ISA_8bit, U1 8088, U10 8288, U11 74LS126, U2 74LS573, U3 74LS573, U4 74LS245, U5 82188, U6 8284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

Commit message: update 8088 max
Parts:
- removed R4, R5, R6: 10K ohm, Resistor_THT:R_Axial_DIN0207_L6.3mm_D2.5mm_P10.16mm_Horizontal
- added RN1: 10K ohm, Resistor_THT:R_Array_SIP9, F.Cu at (34.3, 120.6)
- added RN2: 10K ohm, Resistor_THT:R_Array_SIP4, F.Cu at (14.7, 120.6)
Connections:
- U10 pad 11: Net-(U10-Pad11) -> /IOWR
- U10 pad 12: /IORD -> Net-(U10-Pad12)
- U10 pad 13: /IOWR -> /IORD
- U10 pad 16: /DEN -> Net-(U10-Pad16)
- U10 pad 7: /MWR -> /MRD
- U10 pad 8: /MRD -> Net-(U10-Pad8)
- U10 pad 9: Net-(U10-Pad9) -> /MWR
- U4 pad 19: /DEN -> /HOLDA
Routing:
- net /TEST: track 154.8 -> 38.6 mm, vias 4 -> 1
- net /DEN: track 74.4 -> 0.00 mm, vias 3 -> 0
- net /S2: track 106.6 -> 144.2 mm, vias 3 -> 4
- net /5+: track 577.3 -> 613.1 mm
- net /8087_INT: track 52.3 -> 87.9 mm, vias 2 -> 3
- net /HOLDA: track 206.3 -> 241.6 mm, vias 11 -> 13
- net /RQ_8087: track 21.4 -> 56.4 mm, vias 0 -> 1
- net /S1: track 117.9 -> 150.3 mm, vias 3 -> 4
- net /RQ_82188: track 95.0 -> 122.9 mm, vias 4 -> 5
- net /S0: track 113.5 -> 140.9 mm, vias 3 -> 4
- net /IOWR: track 125.9 -> 140.2 mm, vias 4 -> 6
- net /RESET: track 174.7 -> 179.8 mm
- net /NMI: track 111.2 -> 114.5 mm, vias 3 -> 4
- net /MWR: track 86.9 -> 90.2 mm, vias 2 -> 4
- net /MRD: track 85.5 -> 82.9 mm
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