File: Kicad/8088 MAX ISA/8088.sch (KiCad schematic (older format))
At the start: 31 parts, among them J1 Conn_02x08_Counter_Clockwise, J9 Bus_ISA_8bit, U1 8088, U10 8288, U11 74LS126, U2 74LS573, U3 74LS573, U4 74LS245, U5 82188, U6 8284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

Commit message: update 8088 max
Parts:
- removed R4, R5, R6: 10K ohm, Resistor_THT:R_Axial_DIN0207_L6.3mm_D2.5mm_P10.16mm_Horizontal, symbol Device:R
- added RN1: 10K ohm, Resistor_THT:R_Array_SIP9, symbol Device:R_Network08
- added RN2: 10K ohm, Resistor_THT:R_Array_SIP4, symbol Device:R_Network03
Connections:
- net 5+: now also RN1.1 (common)
- net 8087_INT: now also RN2.3 (R2)
- net 8088_NMI: now also RN2.2 (R1)
- net GND: now also RN2.1 (common)
- net HOLDA: now also U4.19 (CE)
- net IORD: now also U10.13 (~IORC~); no longer U10.12 (~AIOWC~)
- net IOWR: now also U10.11 (~IOWC~); no longer U10.13 (~IORC~)
- net MRD: now also U10.7 (~MRDC~); no longer U10.8 (~AMWC~)
- net MWR: now also U10.9 (~MWTC~); no longer U10.7 (~MRDC~)
- net NMI: now also RN2.4 (R3)
- net RQ_8087: now also RN1.6 (R5)
- net RQ_82188: now also RN1.7 (R6)
- net S0: now also RN1.4 (R3)
- net S1: now also RN1.3 (R2)
- net S2: now also RN1.2 (R1)
- net TEST: now also RN1.5 (R4)
- net DEN: no longer names the net of U10.16 (DEN)
- net DEN: no longer U4.19 (CE)
Changed lines of the file:
@@
 Text Label 4625 7250 2    50   ~ 0
 HOLD
-Text Label 8825 6900 0    50   ~ 0
-IORD
-Text Label 8825 7000 0    50   ~ 0
-MRD
-Text Label 8825 7300 0    50   ~ 0
-MWR
-Text Label 8825 7400 0    50   ~ 0
-IOWR
 Text Label 8825 7800 0    50   ~ 0
 DTR
-Text Label 8825 8100 0    50   ~ 0
-DEN
-Text Label 11575 8750 2    50   ~ 0
-DEN
 Text Label 11575 8650 2    50   ~ 0
 DTR
@@
 Text Label 8825 7900 0    50   ~ 0
 ALE
-Text Label 11200 9100 2    50   ~ 0
-5+
-Text Label 11500 9100 0    50   ~ 0
-DEN
-$Comp
-L Device:R R5
-U 1 1 61072939
-P 11350 9100
-F 0 "R5" V 11143 9100 50  0000 C CNN
-F 1 "10K ohm" V 11234 9100 50  0000 C CNN
-F 2 "Resistor_THT:R_Axial_DIN0207_L6.3mm_D2.5mm_P10.16mm_Horizontal" V 11280 9100 50  0001 C CNN
-F 3 "~" H 11350 9100 50  0001 C CNN
-	1    11350 9100
-	0    1    1    0
-$EndComp
-$Comp
-L 74xx:74LS245 U4
-U 1 1 61063CD3
-P 12075 8250
-F 0 "U4" H 12075 9231 50  0000 C CNN
-F 1 "74LS245" H 12075 9140 50  0000 C CNN
-F 2 "Package_DIP:DIP-20_W7.62mm" H 12075 8250 50  0001 C CNN
-F 3 "http://www.ti.com/lit/gpn/sn74LS245" H 12075 8250 50  0001 C CNN
-	1    12075 8250
-	1    0    0    -1
-$EndComp
 Text Label 7975 13575 0    50   ~ 0
 SPK_GO
@@
 	1    0    0    -1
 $EndComp
-Text Label 7425 7700 2    50   ~ 0
-HOLDA
 Text Label 8050 5800 0    50   ~ 0
 GND
@@
 	1    0    0    -1
 $EndComp
-Text Label 7425 7900 2    50   ~ 0
-GND
-Text Label 7425 6900 2    50   ~ 0
-S0
-Text Label 7425 7000 2    50   ~ 0
-S1
-Text Label 7425 7100 2    50   ~ 0
-S2
 Text Label 8650 5100 0    50   ~ 0
 S0
@@
 Text Label 5950 5400 0    50   ~ 0
 8087_INT
-$Comp
-L Device:R R4
-U 1 1 6325BF49
-P 2400 8025
-F 0 "R4" V 2193 8025 50  0000 C CNN
-F 1 "10K ohm" V 2284 8025 50  0000 C CNN
-F 2 "Resistor_THT:R_Axial_DIN0207_L6.3mm_D2.5mm_P10.16mm_Horizontal" V 2330 8025 50  0001 C CNN
-F 3 "~" H 2400 8025 50  0001 C CNN
-	1    2400 8025
-	0    1    1    0
-$EndComp
-Text Label 2250 8025 2    50   ~ 0
-GND
-Text Label 2550 8025 0    50   ~ 0
+Text Label 1075 7650 2    50   ~ 0
+GND
+Text Label 1475 7650 0    50   ~ 0
 8088_NMI
 Text Label 3250 6075 0    50   ~ 0
@@
 Text Label 7250 3200 2    50   ~ 0
 8088_NMI
-$Comp
-L Device:R R6
-U 1 1 632AB08C
-P 6725 3650
-F 0 "R6" V 6518 3650 50  0000 C CNN
-F 1 "10K ohm" V 6609 3650 50  0000 C CNN
-F 2 "Resistor_THT:R_Axial_DIN0207_L6.3mm_D2.5mm_P10.16mm_Horizontal" V 6655 3650 50  0001 C CNN
-F 3 "~" H 6725 3650 50  0001 C CNN
-	1    6725 3650
-	0    1    1    0
-$EndComp
-Text Label 6575 3650 2    50   ~ 0
-5+
-Text Label 6875 3650 0    50   ~ 0
-TEST
 Text Label 5950 5300 0    50   ~ 0
 TEST
 Text Label 7250 3700 2    50   ~ 0
 TEST
+Text Label 6400 7250 2    50   ~ 0
+5+
+Text Label 7425 7100 2    50   ~ 0
+S2
+Text Label 7425 7000 2    50   ~ 0
+S1
+Text Label 7425 6900 2    50   ~ 0
+S0
+Text Label 6800 7250 0    50   ~ 0
+S2
+Text Label 6800 7150 0    50   ~ 0
+S1
+Text Label 6800 7050 0    50   ~ 0
+S0
+Text Label 7425 7900 2    50   ~ 0
+GND
+$Comp
+L 74xx:74LS245 U4
+U 1 1 61063CD3
+P 12075 8250
+F 0 "U4" H 12075 9231 50  0000 C CNN
+F 1 "74LS245" H 12075 9140 50  0000 C CNN
+F 2 "Package_DIP:DIP-20_W7.62mm" H 12075 8250 50  0001 C CNN
+F 3 "http://www.ti.com/lit/gpn/sn74LS245" H 12075 8250 50  0001 C CNN
+	1    12075 8250
+	1    0    0    -1
+$EndComp
+Text Label 11575 8750 2    50   ~ 0
+HOLDA
+Text Label 6800 6850 0    50   ~ 0
+RQ_8087
+Text Label 6800 6750 0    50   ~ 0
+RQ_82188
+Text Label 6800 6950 0    50   ~ 0
+TEST
+$Comp
+L Device:R_Network08 RN1
+U 1 1 633537E3
+P 6600 6850
+F 0 "RN1" V 6925 6850 50  0000 C CNN
+F 1 "10K ohm" V 6834 6850 50  0000 C CNN
+F 2 "Resistor_THT:R_Array_SIP9" V 7175 6850 50  0001 C CNN
+F 3 "http://www.vishay.com/docs/31509/csc.pdf" H 6600 6850 50  0001 C CNN
+	1    6600 6850
+	0    -1   -1   0
+$EndComp
+$Comp
+L Device:R_Network03 RN2
+U 1 1 6325F6F1
+P 1275 7550
+F 0 "RN2" V 1600 7550 50  0000 C CNN
+F 1 "10K ohm" V 1509 7550 50  0000 C CNN
+F 2 "Resistor_THT:R_Array_SIP4" V 1850 7550 50  0001 C CNN
+F 3 "http://www.vishay.com/docs/31509/csc.pdf" H 1275 7550 50  0001 C CNN
+	1    1275 7550
+	0    -1   -1   0
+$EndComp
+Text Label 1475 7550 0    50   ~ 0
+8087_INT
+Text Label 1475 7450 0    50   ~ 0
+NMI
+Text Label 8825 7400 0    50   ~ 0
+IORD
+Text Label 8825 7300 0    50   ~ 0
+MRD
+Text Label 8825 7200 0    50   ~ 0
+MWR
+Text Label 8825 7100 0    50   ~ 0
+IOWR
+Text Label 7425 7700 2    50   ~ 0
+HOLDA
 $EndSCHEMATC
