File: Kicad/Breadboard Adapter/Breadboard Adapter.kicad_pcb (KiCad board)
At the start: 2 copper layers, 20.6 x 137.2 mm, 11 parts, among them J1 Conn_02x08_Counter_Clockwise, J2 USB_C_Receptacle_USB2.0, J3 Conn_01x31, J4 Conn_01x31, J5 Conn_01x8, J6 Conn_01x8, J9 Bus_ISA_8bit, SW1 SW_Push_DPDT

Commit message: updates
Parts:
- moved C1 1.50 mm to (109.2, 146.8), turned to 180 degrees
Connections:
- C1 pad 1: /GND -> /RESET
- C1 pad 2: /RESET -> /GND
