File: Kicad/8088 ISA/8088.sch (KiCad schematic (older format))
At the start: 24 parts, among them J1 Conn_02x08_Counter_Clockwise, J9 Bus_ISA_8bit, U1 8284, U2 74LS573, U3 74LS573, U4 74LS245, U5 8088, U6 8259, U7 8253, U8 74LS257, Y1 Crystal

Commit message: update 8088 card
Parts:
- renumbered R2 to R1, R4 to R2, R5 to R4, R1 to R5, U5 to U1, U3 to U2, U2 to U3, U8 to U5, U1 to U6, U6 to U7, U7 to U8
Other:
- moved on the sheet: C5, C6, C8
Changed lines of the file:
@@
 $EndComp
 $Comp
-L 74xx:74LS573 U3
+L 74xx:74LS573 U2
 U 1 1 610632BC
 P 12075 3450
-F 0 "U3" H 12075 4431 50  0000 C CNN
+F 0 "U2" H 12075 4431 50  0000 C CNN
 F 1 "74LS573" H 12075 4340 50  0000 C CNN
 F 2 "Package_DIP:DIP-20_W7.62mm" H 12075 3450 50  0001 C CNN
@@
 $EndComp
 $Comp
-L 74xx:74LS573 U2
+L 74xx:74LS573 U3
 U 1 1 610661C4
 P 12050 5925
-F 0 "U2" H 12050 6906 50  0000 C CNN
+F 0 "U3" H 12050 6906 50  0000 C CNN
 F 1 "74LS573" H 12050 6815 50  0000 C CNN
 F 2 "Package_DIP:DIP-20_W7.62mm" H 12050 5925 50  0001 C CNN
@@
 DEN
 $Comp
-L Device:R R1
+L Device:R R5
 U 1 1 61072939
 P 11350 9100
-F 0 "R1" V 11143 9100 50  0000 C CNN
+F 0 "R5" V 11143 9100 50  0000 C CNN
 F 1 "10K ohm" V 11234 9100 50  0000 C CNN
 F 2 "Resistor_THT:R_Axial_DIN0207_L6.3mm_D2.5mm_P10.16mm_Horizontal" V 11280 9100 50  0001 C CNN
@@
 X2
 $Comp
-L Device:R R4
+L Device:R R2
 U 1 1 610DFCED
 P 3400 4050
-F 0 "R4" V 3193 4050 50  0000 C CNN
+F 0 "R2" V 3193 4050 50  0000 C CNN
 F 1 "510 ohm" V 3284 4050 50  0000 C CNN
 F 2 "Resistor_THT:R_Axial_DIN0207_L6.3mm_D2.5mm_P10.16mm_Horizontal" V 3330 4050 50  0001 C CNN
@@
 X1
 $Comp
-L MCU_Intel:8088 U5
+L MCU_Intel:8088 U1
 U 1 1 6113D842
 P 7750 3825
-F 0 "U5" H 7750 5806 50  0000 C CNN
+F 0 "U1" H 7750 5806 50  0000 C CNN
 F 1 "8088" H 7750 5715 50  0000 C CNN
 F 2 "Package_DIP:DIP-40_W15.24mm" H 7800 3925 50  0001 C CIN
@@
 $EndComp
 $Comp
-L Interface:8259 U6
+L Interface:8259 U7
 U 1 1 6113F110
 P 7775 7725
-F 0 "U6" H 7775 9006 50  0000 C CNN
+F 0 "U7" H 7775 9006 50  0000 C CNN
 F 1 "8259" H 7775 8915 50  0000 C CNN
 F 2 "Package_DIP:DIP-28_W15.24mm" H 7775 7725 50  0001 C CIN
@@
 $EndComp
 $Comp
-L Timer:8253 U7
+L Timer:8253 U8
 U 1 1 6114018C
 P 7775 10700
-F 0 "U7" H 7775 11881 50  0000 C CNN
+F 0 "U8" H 7775 11881 50  0000 C CNN
 F 1 "8253" H 7775 11790 50  0000 C CNN
 F 2 "Package_DIP:DIP-24_W15.24mm" H 7825 10950 50  0001 C CNN
@@
 $EndComp
 $Comp
-L Timer:8284 U1
+L Timer:8284 U6
 U 1 1 61142859
 P 2100 3500
-F 0 "U1" H 2100 4581 50  0000 C CNN
+F 0 "U6" H 2100 4581 50  0000 C CNN
 F 1 "8284" H 2100 4490 50  0000 C CNN
 F 2 "Package_DIP:DIP-18_W7.62mm" H 2100 3500 50  0001 C CIN
@@
 RD
 $Comp
-L Device:R R5
+L Device:R R4
 U 1 1 61146C76
 P 11875 10025
-F 0 "R5" V 11668 10025 50  0000 C CNN
+F 0 "R4" V 11668 10025 50  0000 C CNN
 F 1 "10K ohm" V 11759 10025 50  0000 C CNN
 F 2 "Resistor_THT:R_Axial_DIN0207_L6.3mm_D2.5mm_P10.16mm_Horizontal" V 11805 10025 50  0001 C CNN
@@
 CLK1
 $Comp
-L Device:R R2
+L Device:R R1
 U 1 1 6115385B
 P 3325 2725
-F 0 "R2" V 3118 2725 50  0000 C CNN
+F 0 "R1" V 3118 2725 50  0000 C CNN
 F 1 "27 ohm" V 3209 2725 50  0000 C CNN
 F 2 "Resistor_THT:R_Axial_DIN0207_L6.3mm_D2.5mm_P10.16mm_Horizontal" V 3255 2725 50  0001 C CNN
@@
 READY1
 $Comp
-L 74xx:74LS257 U8
+L 74xx:74LS257 U5
 U 1 1 6114181C
 P 12050 11500
-F 0 "U8" H 12050 12581 50  0000 C CNN
+F 0 "U5" H 12050 12581 50  0000 C CNN
 F 1 "74LS257" H 12050 12490 50  0000 C CNN
 F 2 "Package_DIP:DIP-16_W7.62mm" H 12050 11500 50  0001 C CNN
@@
 	0    1    1    0
 $EndComp
-Text Label 6825 9475 0    50   ~ 0
-GND
-Text Label 6325 9475 2    50   ~ 0
+Text Label 1725 1925 0    50   ~ 0
+GND
+Text Label 1225 1925 2    50   ~ 0
 5+
 $Comp
 L pspice:CAP C6
 U 1 1 61169247
-P 6575 9475
-F 0 "C6" V 6260 9475 50  0000 C CNN
-F 1 "0.1uF" V 6351 9475 50  0000 C CNN
-F 2 "Capacitor_THT:C_Disc_D4.3mm_W1.9mm_P5.00mm" H 6575 9475 50  0001 C CNN
-F 3 "~" H 6575 9475 50  0001 C CNN
-	1    6575 9475
-	0    1    1    0
-$EndComp
-Text Label 11400 10550 0    50   ~ 0
+P 1475 1925
+F 0 "C6" V 1160 1925 50  0000 C CNN
+F 1 "0.1uF" V 1251 1925 50  0000 C CNN
+F 2 "Capacitor_THT:C_Disc_D4.3mm_W1.9mm_P5.00mm" H 1475 1925 50  0001 C CNN
+F 3 "~" H 1475 1925 50  0001 C CNN
+	1    1475 1925
+	0    1    1    0
+$EndComp
+Text Label 8700 9425 0    50   ~ 0
 GND
 $Comp
 L pspice:CAP C8
 U 1 1 61169660
-P 11150 10550
-F 0 "C8" V 10835 10550 50  0000 C CNN
-F 1 "0.1uF" V 10926 10550 50  0000 C CNN
-F 2 "Capacitor_THT:C_Disc_D4.3mm_W1.9mm_P5.00mm" H 11150 10550 50  0001 C CNN
-F 3 "~" H 11150 10550 50  0001 C CNN
-	1    11150 10550
-	0    1    1    0
-$EndComp
-Text Label 10900 10550 2    50   ~ 0
-5+
-Text Label 2750 2275 0    50   ~ 0
-GND
-Text Label 2250 2275 2    50   ~ 0
+P 8450 9425
+F 0 "C8" V 8135 9425 50  0000 C CNN
+F 1 "0.1uF" V 8226 9425 50  0000 C CNN
+F 2 "Capacitor_THT:C_Disc_D4.3mm_W1.9mm_P5.00mm" H 8450 9425 50  0001 C CNN
+F 3 "~" H 8450 9425 50  0001 C CNN
+	1    8450 9425
+	0    1    1    0
+$EndComp
+Text Label 8200 9425 2    50   ~ 0
+5+
+Text Label 12775 10250 0    50   ~ 0
+GND
+Text Label 12275 10250 2    50   ~ 0
 5+
 $Comp
 L pspice:CAP C5
 U 1 1 6116A3B9
-P 2500 2275
-F 0 "C5" V 2185 2275 50  0000 C CNN
-F 1 "0.1uF" V 2276 2275 50  0000 C CNN
-F 2 "Capacitor_THT:C_Disc_D4.3mm_W1.9mm_P5.00mm" H 2500 2275 50  0001 C CNN
-F 3 "~" H 2500 2275 50  0001 C CNN
-	1    2500 2275
-	0    1    1    0
-$EndComp
+P 12525 10250
+F 0 "C5" V 12210 10250 50  0000 C CNN
+F 1 "0.1uF" V 12301 10250 50  0000 C CNN
+F 2 "Capacitor_THT:C_Disc_D4.3mm_W1.9mm_P5.00mm" H 12525 10250 50  0001 C CNN
+F 3 "~" H 12525 10250 50  0001 C CNN
+	1    12525 10250
+	0    1    1    0
+$EndComp

Commit message: Updated Gerber's
Connections:
- net DRQ0: now also U8.13 (OUT1)
Changed lines of the file:
@@
 Text Label 7050 2525 2    50   ~ 0
 READY1
+Text Label 8375 10800 0    50   ~ 0
+DRQ0
 $EndSCHEMATC
