File: Kicad/V40 64K 640K ISA/V40 64K 640K ISA.kicad_pcb (KiCad board)
At the start: 2 copper layers, 165.1 x 73.9 mm, 29 parts, among them J1 Conn_02x08_Counter_Clockwise, J9 Bus_ISA_8bit, U1 64K ROM, U10 74LS573, U2 64K, U3 AS6C1008, U4 AS6C4008, U5 74LS139, U6 74LS138, U7 70208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

Commit message: updates
Parts:
- moved R2 142.5 mm to (173.0, 58.6), turned to 90 degrees
- moved U9 139.8 mm to (165.9, 47.2), turned to 270 degrees
- moved C9 138.3 mm to (169.2, 49.8), turned to 270 degrees
- moved U8 118.7 mm to (135.4, 47.2), turned to 270 degrees
- moved C8 117.5 mm to (138.7, 49.8), turned to 270 degrees
- moved U10 76.7 mm to (104.9, 47.2), turned to 270 degrees
- moved C10 73.3 mm to (108.2, 49.8), turned to 270 degrees
- moved Y1 62.1 mm to (63.5, 103.6), turned to 180 degrees
- moved R1 35.8 mm to (53.8, 109.7), turned to 0 degrees
- moved C7 27.7 mm to (77.5, 79.3), turned to 270 degrees
- moved U7 21.7 mm to (72.6, 84.3), turned to 270 degrees
Connections:
- R pad 1: /GND -> GND
- R pad 1: (no net) -> GND
Routing:
- net /A16: track 247.3 -> 149.7 mm, vias 9 -> 5
- net /DTR: track 60.9 -> 155.7 mm, vias 2 -> 4
- net /AD7: track 44.5 -> 138.3 mm, vias 1 -> 3
- net /AD5: track 44.4 -> 134.8 mm, vias 1 -> 3
- net /DEN: track 71.8 -> 161.7 mm, vias 3 -> 6
- net /AD4: track 41.6 -> 129.9 mm, vias 1 -> 3
- net /A18: track 268.3 -> 181.8 mm, vias 9 -> 8
- net /AD0: track 48.7 -> 132.2 mm, vias 1 -> 3
- net /AD1: track 50.9 -> 134.3 mm, vias 1 -> 3
- net /AD2: track 47.5 -> 130.2 mm, vias 1 -> 3
- net /AD3: track 53.5 -> 132.3 mm, vias 2 -> 3
- net /AD6: track 58.0 -> 135.3 mm, vias 1 -> 3
- net /A19: track 220.2 -> 149.3 mm, vias 8 -> 6
- net VCC: track 462.1 -> 393.3 mm, vias 16 -> 13
- net /A17: track 230.7 -> 175.1 mm
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Other:
- board size 165.1 x 73.9 mm -> 145.8 x 91.4 mm
- board text added: "EMM COMPUTERS V40, 640K RAM, 64K ROM Copyright (C) 2023 EMM www.homebrew8088.com"
- board text removed: "EMM COMPUTERS V40, 640K RAM, 64K ROM Copyright (C) 2022 EMM www.homebrew8088.com"

Commit message: Updated Gerber's
Connections:
- U7 pad 36: Net-(U7-Pad36) -> /DRQ0
- U7 pad 5: /REFRQ -> Net-(U7-Pad5)
Routing:
- net /REFRQ: track 92.7 -> 0.00 mm, vias 4 -> 0
- net /DRQ0: track 0.00 -> 62.5 mm, vias 0 -> 4
