File: Kicad/V40 64K 640K ISA/V40 64K 640K ISA.sch (KiCad schematic (older format))
At the start: 25 parts, among them J1 Conn_02x08_Counter_Clockwise, J9 Bus_ISA_8bit, U1 64K ROM, U10 74LS573, U2 64K, U3 AS6C1008, U4 AS6C4008, U5 74LS139, U6 74LS138, U7 70208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

Commit message: Updated Gerber's
Connections:
- net DRQ0: now also U7.36 (INTAK/SRDY/TOUT1)
- net REFRQ: no longer U7.5 (REFRQ)
Changed lines of the file:
@@
 Text Label 2525 5975 1    50   ~ 0
 A16_
-Text Label 2925 5975 1    50   ~ 0
-REFRQ
 Text Label 3325 5975 1    50   ~ 0
 5+
@@
 Text Label 6625 10175 0    50   ~ 0
 GND
+Text Label 3425 8375 3    50   ~ 0
+DRQ0
 $EndSCHEMATC
