File: Kicad/V40 ISA/V40.kicad_pcb (KiCad board)
At the start: 2 copper layers, 132 x 73.9 mm, 17 parts, among them J1 Conn_02x08_Counter_Clockwise, J9 Bus_ISA_8bit, U1 70208, U2 74LS573, U3 74LS573, U4 74LS245, Y1 Crystal

Commit message: updates
Other:
- board text added: "EMM COMPUTERS V40 (70208) PROCESSOR, NO DMA Copyright (C) 2022 EMM www.homebrew8088.com"
- board text removed: "EMM COMPUTERS V40 (70208) PROCESSOR, NO DMA Copyright (C) 2021 EMM www.homebrew8088.com"

Commit message: Updated Gerber's
Connections:
- U1 pad 36: Net-(U1-Pad36) -> /DRQ0
- U1 pad 5: /REFRQ -> Net-(U1-Pad5)
Routing:
- net /DRQ0: track 0.00 -> 103.5 mm, vias 0 -> 3
- net /REFRQ: track 102.6 -> 0.00 mm, vias 3 -> 0
Other:
- board text added: "EMM COMPUTERS V40 (70208) PROCESSOR, NO DMA Copyright (C) 2023 EMM www.homebrew8088.com"
- board text removed: "EMM COMPUTERS V40 (70208) PROCESSOR, NO DMA Copyright (C) 2022 EMM www.homebrew8088.com"
