File: Kicad/V40 ISA/V40.sch (KiCad schematic (older format))
At the start: 13 parts, among them J1 Conn_02x08_Counter_Clockwise, J9 Bus_ISA_8bit, U1 70208, U2 74LS573, U3 74LS573, U4 74LS245, Y1 Crystal

Commit message: Updated Gerber's
Connections:
- net DRQ0: now also U1.36 (INTAK/SRDY/TOUT1)
- net REFRQ: no longer U1.5 (REFRQ)
Changed lines of the file:
@@
 Text Label 17925 7275 0    50   ~ 0
 RESET
-Text Label 7625 3575 1    50   ~ 0
-REFRQ
 Text Label 7825 3575 1    50   ~ 0
 HOLDA
@@
 Text Label 8225 3575 1    50   ~ 0
 RDY1
+Text Label 8125 5975 3    50   ~ 0
+DRQ0
 $EndSCHEMATC
