File: Kicad/Multi ATX ISA With DMA/Multi.kicad_pcb (KiCad board)
At the start: 2 copper layers, 182.9 x 172.7 mm, 118 parts, among them J1 Bus_ISA_8bit, J10 Conn_02x08_Counter_Clockwise, J11 Bus_ISA_8bit, J2 Mini-DIN-6, J3 SPK, J4 Bus_ISA_8bit, J5 Bus_ISA_8bit, J6 PWR ON, J7 Bus_ISA_8bit, J8 Bus_ISA_8bit, J9 Bus_ISA_8bit, SW1 RESET, U1 74LS139, U11 8284, U117 74LS139, U12 74LS138, U13 74LS138, U14 74LS74, U15 74LS573, U16 74LS04, U17 74LS139, U19 82C42/83C42, U2 74LS245, U20 74LS07, U3 33 ohm, U61 8237, U63 74LS04, U64 74LS670, U65 74LS573, U9 74LS138, Y2 14.31818 MHz

Commit message: Updated Gerber's
Parts:
- added J12: RESET, Connector_PinHeader_2.54mm:PinHeader_1x02_P2.54mm_Vertical, F.Cu at (126.0, 161.0)
- added SW2: DRQ0/DACK0 EN, Package_DIP:DIP-4_W7.62mm, F.Cu at (9.91, 140.5)
- U19: value 82C42/83C42 -> 82C42
Routing:
- net /DRQ0_: track 3.36 -> 99.1 mm, vias 0 -> 3
- net /DRQ0: track 37.6 -> 128.1 mm, vias 0 -> 6
- net /DACK0: track 0.00 -> 75.2 mm, vias 0 -> 4
- net /REFRQ: track 186.5 -> 244.7 mm, vias 1 -> 3
- net /RESET: track 323.3 -> 330.3 mm
- net /GND: track 1567.9 -> 1574.3 mm
- net /HOLD: track 187.0 -> 186.4 mm

Commit message: ADDED Port
Parts:
- SW2: footprint Package_DIP:DIP-4_W7.62mm -> Button_Switch_THT:SW_DIP_SPSTx02_Slide_9.78x7.26mm_W7.62mm_P2.54mm
