File: Kicad/Multi ATX ISA With DMA/Multi.sch (KiCad schematic (older format))
At the start: 85 parts, among them J1 Bus_ISA_8bit, J10 Conn_02x08_Counter_Clockwise, J11 Bus_ISA_8bit, J2 Mini-DIN-6, J3 SPK, J4 Bus_ISA_8bit, J5 Bus_ISA_8bit, J6 PWR ON, J7 Bus_ISA_8bit, J8 Bus_ISA_8bit, J9 Bus_ISA_8bit, SW1 RESET, U1 74LS139, U11 8284, U117 74LS139, U12 74LS138, U13 74LS138, U14 74LS74, U15 74LS573, U16 74LS04, U17 74LS139, U19 82C42/83C42, U2 74LS245, U20 74LS07, U3 33 ohm, U61 8237, U63 74LS04, U64 74LS670, U65 74LS573, U9 74LS138, Y2 14.31818 MHz

Commit message: Updated Gerber's
Parts:
- added J12: RESET, Connector_PinHeader_2.54mm:PinHeader_1x02_P2.54mm_Vertical, symbol Connector_Generic:Conn_01x02
- added SW2: DRQ0/DACK0 EN, Package_DIP:DIP-4_W7.62mm, symbol Switch:SW_DIP_x02
- U19: value 82C42/83C42 -> 82C42
Connections:
- net DACK0: now also SW2.2
- net DRQ0: now also SW2.4
- net DRQ0_: now also SW2.1
- net GND: now also J12.2 (Pin_2)
- net REFRQ: now also SW2.3
- net RESET: now also J12.1 (Pin_1)
Changed lines of the file:
@@
 P 8300 9950
 F 0 "U19" H 8300 10015 50  0000 C CNN
-F 1 "82C42/83C42" H 8300 9924 50  0000 C CNN
+F 1 "82C42" H 8300 9924 50  0000 C CNN
 F 2 "Package_LCC:PLCC-44_THT-Socket" H 8300 9950 50  0001 C CNN
 F 3 "" H 8300 9950 50  0001 C CNN
@@
 Text Label 17450 2850 2    50   ~ 0
 5+
+$Comp
+L Switch:SW_DIP_x02 SW2
+U 1 1 63F01F95
+P 15850 9200
+F 0 "SW2" H 15850 9567 50  0000 C CNN
+F 1 "DRQ0/DACK0 EN" H 15850 9476 50  0000 C CNN
+F 2 "Package_DIP:DIP-4_W7.62mm" H 15850 9200 50  0001 C CNN
+F 3 "~" H 15850 9200 50  0001 C CNN
+	1    15850 9200
+	1    0    0    -1
+$EndComp
+Text Label 15550 9100 2    50   ~ 0
+DRQ0_
+Text Label 15550 9200 2    50   ~ 0
+DACK0
+Text Label 16150 9200 0    50   ~ 0
+REFRQ
+Text Label 16150 9100 0    50   ~ 0
+DRQ0
+$Comp
+L Connector_Generic:Conn_01x02 J12
+U 1 1 63F7D6D0
+P 2150 6225
+F 0 "J12" H 2230 6217 50  0001 L CNN
+F 1 "RESET" H 2230 6171 50  0000 L CNN
+F 2 "Connector_PinHeader_2.54mm:PinHeader_1x02_P2.54mm_Vertical" H 2150 6225 50  0001 C CNN
+F 3 "~" H 2150 6225 50  0001 C CNN
+	1    2150 6225
+	1    0    0    -1
+$EndComp
+Text Label 1950 6325 2    50   ~ 0
+GND
+Text Label 1950 6225 2    50   ~ 0
+RESET
 $EndSCHEMATC

Commit message: ADDED Port
Parts:
- SW2: footprint Package_DIP:DIP-4_W7.62mm -> Button_Switch_THT:SW_DIP_SPSTx02_Slide_9.78x7.26mm_W7.62mm_P2.54mm
Changed lines of the file:
@@
 F 0 "SW2" H 15850 9567 50  0000 C CNN
 F 1 "DRQ0/DACK0 EN" H 15850 9476 50  0000 C CNN
-F 2 "Package_DIP:DIP-4_W7.62mm" H 15850 9200 50  0001 C CNN
+F 2 "Button_Switch_THT:SW_DIP_SPSTx02_Slide_9.78x7.26mm_W7.62mm_P2.54mm" H 15850 9200 50  0001 C CNN
 F 3 "~" H 15850 9200 50  0001 C CNN
 	1    15850 9200
